File: v1/ac-monitor.kicad_sch (KiCad schematic)
At the start: 3 parts, among them U6 MID400

Commit message: cleanups
Changed lines of the file:
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@@
     (stroke (width 0) (type solid) (color 0 0 0 0))
   )
-  (wire (pts (xy 103.505 57.15) (xy 103.505 60.96))
+  (wire (pts (xy 103.505 59.055) (xy 103.505 60.96))
     (stroke (width 0) (type solid) (color 0 0 0 0))
   )
@@
     (stroke (width 0) (type solid) (color 0 0 0 0))
   )
-  (wire (pts (xy 120.015 55.88) (xy 120.015 61.1632))
+  (wire (pts (xy 120.015 59.055) (xy 120.015 61.1632))
     (stroke (width 0) (type solid) (color 0 0 0 0))
   )
@@
     )
   )
-  (symbol (lib_id "power:+5V") (at 103.505 57.15 0)
+  (symbol (lib_id "power:+5V") (at 103.505 59.055 0)
     (in_bom yes) (on_board yes)
-    (property "Reference" "#PWR038" (id 0) (at 103.505 60.96 0)
+    (property "Reference" "#PWR038" (id 0) (at 103.505 62.865 0)
       (effects (font (size 1.27 1.27)) hide)
     )
-    (property "Value" "+5V" (id 1) (at 103.8733 52.8256 0))
-    (property "Footprint" "" (id 2) (at 103.505 57.15 0)
+    (property "Value" "+5V" (id 1) (at 103.8733 54.7306 0))
+    (property "Footprint" "" (id 2) (at 103.505 59.055 0)
       (effects (font (size 1.27 1.27)) hide)
     )
-    (property "Datasheet" "" (id 3) (at 103.505 57.15 0)
+    (property "Datasheet" "" (id 3) (at 103.505 59.055 0)
       (effects (font (size 1.27 1.27)) hide)
     )
   )
-  (symbol (lib_id "power:VCC") (at 120.015 55.88 0)
+  (symbol (lib_id "power:VCC") (at 120.015 59.055 0)
     (in_bom yes) (on_board yes)
-    (property "Reference" "#PWR040" (id 0) (at 120.015 59.69 0)
+    (property "Reference" "#PWR040" (id 0) (at 120.015 62.865 0)
       (effects (font (size 1.27 1.27)) hide)
     )
-    (property "Value" "VCC" (id 1) (at 120.396 51.4858 0))
-    (property "Footprint" "" (id 2) (at 120.015 55.88 0)
+    (property "Value" "VCC" (id 1) (at 120.396 54.6608 0))
+    (property "Footprint" "" (id 2) (at 120.015 59.055 0)
       (effects (font (size 1.27 1.27)) hide)
     )
-    (property "Datasheet" "" (id 3) (at 120.015 55.88 0)
+    (property "Datasheet" "" (id 3) (at 120.015 59.055 0)
       (effects (font (size 1.27 1.27)) hide)
     )
