File: v1.1/MadPresso.kicad_pcb (KiCad board)
At the start: 2 copper layers, 108 x 57.5 mm, 75 parts, among them J1 Conn_01x07, J2 Conn_01x03, J3 Conn_01x02, J4 Conn_01x04, Q1 BC847, Q2 BSS84, Q3 T835-600B, Q4 2N7002, Q5 T835-600B, Q6 2N7002, Q7 T835-600B, Q8 2N7002, U1 LTV-356T, U2 ADC101C021CIMK, U3 WeMos_D1_mini, U4 MID400, U5 MID400, U6 TLP160G, U7 TLP160G, U8 TLP160G

Commit message: some more documentation
Parts:
- removed REF**: KiCad-Logo2_5mm_Copper, Symbol:KiCad-Logo2_5mm_Copper
- added R32: 360R/0.5W, Resistor_SMD:R_1206_3216Metric_Pad1.30x1.75mm_HandSolder, F.Cu at (38.3, 49.1)
- added R33: 360R/0.5W, Resistor_SMD:R_1206_3216Metric_Pad1.30x1.75mm_HandSolder, F.Cu at (50.1, 43.5)
- added R34: 360R/0.5W, Resistor_SMD:R_1206_3216Metric_Pad1.30x1.75mm_HandSolder, F.Cu at (38.3, 42.1)
Connections:
- R20 pad 2: LINE -> Net-(R20-Pad2)
- R24 pad 2: LINE -> Net-(R24-Pad2)
- R28 pad 2: LINE -> Net-(R28-Pad2)
Routing:
- net LINE: track 5.03 -> 0.00 mm, vias 65 -> 62
- net Net-(R24-Pad2): track 0.00 -> 1.69 mm, vias 0 -> 1
- net Net-(R28-Pad2): track 0.00 -> 1.67 mm, vias 0 -> 1

Commit message: mechanical details for v1.1
Parts:
- removed R32, R33, R34: 360R/0.5W, Resistor_SMD:R_1206_3216Metric_Pad1.30x1.75mm_HandSolder
Connections:
- R20 pad 2: Net-(R20-Pad2) -> LINE
- R24 pad 2: Net-(R24-Pad2) -> LINE
- R28 pad 2: Net-(R28-Pad2) -> LINE
Routing:
- net LINE: track 0.00 -> 5.03 mm, vias 62 -> 65
- net Net-(R24-Pad2): track 1.69 -> 0.00 mm, vias 1 -> 0
- net Net-(R28-Pad2): track 1.67 -> 0.00 mm, vias 1 -> 0

Commit message: v1.1a
Parts:
- added REF**: OSHW-Logo2_7.3x6mm_SilkScreen, Symbol:OSHW-Logo2_7.3x6mm_SilkScreen, F.Cu at (92.7, 53.8)
Other:
- board text added: "MadPresso v1.1a"
- board text removed: "MadPresso v1.1"
